Commit message: Fixed LIDAR plugin

File: urdf/hykabai.urdf (robot description, URDF)
Before this commit: robot hykabai, 4 links, 3 joints
Links:
- added link rplidar_link; collision box size=0.1 0.1 0.1
- link base_link: mass 2.4 -> 1.5
- link left_wheel: mass 0.01 -> 0.0025
- link right_wheel: mass 0.01 -> 0.025
Joints:
- removed joint left_wheel_hinge
- removed joint right_wheel_hinge
- added joint left_wheel_joint: type continuous, parent base_link, child left_wheel, origin xyz=0 -0.09 0.025 rpy=0 0 0, axis 0 1 0, limit effort=100 velocity=100
- added joint lidar_joint: type fixed, parent base_link, child rplidar_link, origin xyz=0 0 0.1 rpy=0 0 0, axis 0 1 0
- added joint right_wheel_joint: type continuous, parent base_link, child right_wheel, origin xyz=0 0.082 0.025 rpy=0 0 0, axis 0 1 0, limit effort=100 velocity=100

Commit message: Added a visualization for mapping configuration

File: urdf/hykabai.urdf (robot description, URDF)
Before this commit: robot hykabai, 5 links, 4 joints
Joints:
- joint lidar_joint: origin xyz=0 0 0.1 rpy=0 0 0 -> xyz=0 0 0 rpy=0 0 0
